File: schematic/el_precheapo.kicad_pcb (KiCad board)
At the start: 2 copper layers, 111.8 x 73.7 mm, 59 parts, among them J1 Conn_01x03, J2 Conn_01x03, J3 Conn_01x02, SW1 SW_SPST, T1 Transformer_1P_SS, U1 L7809, U2 L7909, U3 NE5532, U4 NE5532

Commit message: update to a single volume board mnt version.
Parts:
- removed RV2, RV3, RV4: R_POT, Connector_Molex:Molex_KK-254_AE-6410-03A_1x03_P2.54mm_Vertical
- added R21: 150, Resistor_THT:R_Axial_DIN0207_L6.3mm_D2.5mm_P10.16mm_Horizontal, F.Cu at (152.5, 68.1)
- added R22: 150, Resistor_THT:R_Axial_DIN0207_L6.3mm_D2.5mm_P10.16mm_Horizontal, F.Cu at (143.6, 89.7)
- R1, R2: value 1M -> 100K
- R10, R9: value 1K5 -> 1M_DNP
- RV1: value R_POT -> R_POT_Dual; footprint Connector_Molex:Molex_KK-254_AE-6410-03A_1x03_P2.54mm_Vertical -> Potentiometer_THT:Potentiometer_Alpha_RD902F-40-00D_Dual_Vertical
- moved R9 49.3 mm to (97.9, 66.5), turned to 0 degrees
- moved R10 43.3 mm to (102.5, 99.6), turned to 180 degrees
- moved R8 16.4 mm to (146.8, 79.5), turned to 270 degrees
- moved RV1 4.10 mm to (141.9, 74.3)
Connections:
- R10 pad 1: Net-(R10-Pad1) -> GND
- R10 pad 2: Net-(R10-Pad2) -> Net-(C6-Pad2)
- R8 pad 1: Net-(R10-Pad2) -> Net-(R8-Pad1)
- R9 pad 1: Net-(R7-Pad1) -> Net-(C5-Pad2)
- R9 pad 2: Net-(R9-Pad2) -> GND
- RV1 pad 2: Net-(R9-Pad2) -> Net-(R21-Pad1)
Routing:
- net Net-(C10-Pad1): track 11.9 -> 35.6 mm
- net Net-(R10-Pad1): track 20.8 -> 0.00 mm
- net Net-(R9-Pad2): track 19.0 -> 0.00 mm
- net Net-(R10-Pad2): track 11.9 -> 0.00 mm
- net Net-(R21-Pad1): track 0.00 -> 11.3 mm
- net Net-(C5-Pad2): track 9.59 -> 17.3 mm
- net Net-(R12-Pad2): track 11.8 -> 19.4 mm
- net Net-(C6-Pad2): track 9.08 -> 14.8 mm
- net Net-(R7-Pad1): track 12.2 -> 7.82 mm
- net Net-(R22-Pad2): track 0.00 -> 3.01 mm
- net Net-(R8-Pad1): track 0.00 -> 2.73 mm
- net Net-(R11-Pad1): track 16.5 -> 13.8 mm
- net /power supply/V-: track 115.8 -> 116.7 mm
