File: schematic/preamp.sch (KiCad schematic (older format))
At the start: 46 parts, among them J1 Conn_01x03, J2 Conn_01x03, U3 NE5532, U4 NE5532

Commit message: update to a single volume board mnt version.
Parts:
- removed RV1, RV2, RV3, RV4: R_POT, Connector_Molex:Molex_KK-254_AE-6410-03A_1x03_P2.54mm_Vertical, symbol Device:R_POT
- added R21, R22: 150, Resistor_THT:R_Axial_DIN0207_L6.3mm_D2.5mm_P10.16mm_Horizontal, symbol Device:R
- added RV1: R_POT_Dual, Potentiometer_THT:Potentiometer_Alpha_RD902F-40-00D_Dual_Vertical, symbol Device:R_POT_Dual
- R1, R2: value 1M -> 100K
- R10, R9: value 1K5 -> 1M_DNP
Connections:
- net GND: now also R10.1, R9.2, RV1.3, RV1.4
- net at C5.2, J1.3 (Pin_3): now also R9.1
- net at C6.2, J1.1 (Pin_1): now also R10.2
- net at R7.1: now also RV1.1; no longer R9.1
- net at R8.1: now also RV1.6; no longer R10.2
- net at R12.2, U4.5 (+): now also R22.1
- net at R11.1, U4.3 (+): now also R21.2
- new net: R21.1, RV1.2
- new net: R22.2, RV1.5
Changed lines of the file:
@@
 P 3550 5000
 F 0 "R2" H 3620 5046 50  0000 L CNN
-F 1 "1M" H 3620 4955 50  0000 L CNN
+F 1 "100K" H 3620 4955 50  0000 L CNN
 F 2 "Resistor_THT:R_Axial_DIN0207_L6.3mm_D2.5mm_P10.16mm_Horizontal" V 3480 5000 50  0001 C CNN
 F 3 "~" H 3550 5000 50  0001 C CNN
@@
 P 3550 3900
 F 0 "R1" H 3620 3946 50  0000 L CNN
-F 1 "1M" H 3620 3855 50  0000 L CNN
+F 1 "100K" H 3620 3855 50  0000 L CNN
 F 2 "Resistor_THT:R_Axial_DIN0207_L6.3mm_D2.5mm_P10.16mm_Horizontal" V 3480 3900 50  0001 C CNN
 F 3 "~" H 3550 3900 50  0001 C CNN
@@
 	4800 4700 4800 4800
 Connection ~ 4800 4800
-$Comp
-L Device:R R9
-U 1 1 5FFDDCDB
-P 5650 4050
-F 0 "R9" H 5720 4096 50  0000 L CNN
-F 1 "1K5" H 5720 4005 50  0000 L CNN
-F 2 "Resistor_THT:R_Axial_DIN0207_L6.3mm_D2.5mm_P10.16mm_Horizontal" V 5580 4050 50  0001 C CNN
-F 3 "~" H 5650 4050 50  0001 C CNN
-	1    5650 4050
-	1    0    0    -1
-$EndComp
-$Comp
-L Device:R R10
-U 1 1 5FFDE445
-P 5650 4850
-F 0 "R10" H 5720 4896 50  0000 L CNN
-F 1 "1K5" H 5720 4805 50  0000 L CNN
-F 2 "Resistor_THT:R_Axial_DIN0207_L6.3mm_D2.5mm_P10.16mm_Horizontal" V 5580 4850 50  0001 C CNN
-F 3 "~" H 5650 4850 50  0001 C CNN
-	1    5650 4850
-	1    0    0    -1
-$EndComp
-Wire Wire Line
-	5650 5000 5350 5000
-Wire Wire Line
-	5350 5000 5350 4850
-Wire Wire Line
-	5650 3900 5350 3900
-Wire Wire Line
-	5350 3900 5350 4050
-Wire Wire Line
-	5350 4350 5350 4450
-Wire Wire Line
-	5350 5250 5350 5000
-Connection ~ 5350 5000
-Wire Wire Line
-	5350 3900 5350 3650
-Connection ~ 5350 3900
-Wire Wire Line
-	5650 4700 5950 4700
-Connection ~ 5650 4700
-Wire Wire Line
-	5950 4850 6250 4850
-Wire Wire Line
-	5950 4700 5950 4850
-Wire Wire Line
-	5650 4200 5950 4200
-Wire Wire Line
-	5950 4200 5950 4050
-Wire Wire Line
-	5950 4050 6250 4050
-Connection ~ 5650 4200
 Wire Wire Line
 	6250 4350 6250 4450
-Wire Wire Line
-	5350 4450 6250 4450
-Connection ~ 5350 4450
-Wire Wire Line
-	5350 4450 5350 4550
 Connection ~ 6250 4450
 Wire Wire Line
 	6250 4450 6250 4550
-Wire Wire Line
-	5350 4450 3800 4450
 Connection ~ 3800 4450
 Wire Wire Line
@@
 	1    0    0    -1
 $EndComp
-Wire Wire Line
-	6450 4200 6450 4100
-Wire Wire Line
-	6450 4100 6650 4100
-Wire Wire Line
-	6450 4800 6650 4800
 Wire Wire Line
 	6450 4700 6450 4800
@@
 	6950 4450 6950 4500
 Wire Wire Line
-	6650 4100 6650 3550
+	6650 4100 6650 3800
 Wire Wire Line
 	6650 3550 7300 3550
-Connection ~ 6650 4100
-Wire Wire Line
-	6650 4800 6650 5350
+Wire Wire Line
+	6650 4800 6650 5100
 Wire Wire Line
 	6650 5350 7300 5350
-Connection ~ 6650 4800
 Wire Wire Line
 	7300 3750 6950 3750
@@
 	9550 4450 8800 4450
 Wire Wire Line
-	2350 4450 3550 4450
+	2350 4450 3050 4450
 Wire Wire Line
 	2350 4450 2000 4450
 Connection ~ 2350 4450
 Wire Wire Line
-	3250 3550 2350 3550
+	3250 3550 3050 3550
 Wire Wire Line
 	2350 3550 2350 4350
@@
 	2350 4550 2350 5350
 Wire Wire Line
-	2350 5350 3250 5350
+	2350 5350 3050 5350
 Wire Wire Line
 	3550 5350 4200 5350
@@
 	4800 5250 5050 5250
 Connection ~ 4800 5250
-$Comp
-L Device:R_POT RV2
-U 1 1 60557F32
-P 5350 4700
-F 0 "RV2" H 5281 4746 50  0000 R CNN
-F 1 "R_POT" H 5281 4655 50  0000 R CNN
-F 2 "Connector_Molex:Molex_KK-254_AE-6410-03A_1x03_P2.54mm_Vertical" H 5350 4700 50  0001 C CNN
-F 3 "~" H 5350 4700 50  0001 C CNN
-	1    5350 4700
-	1    0    0    -1
-$EndComp
-$Comp
-L Device:R_POT RV1
-U 1 1 605586CF
-P 5350 4200
-F 0 "RV1" H 5281 4246 50  0000 R CNN
-F 1 "R_POT" H 5281 4155 50  0000 R CNN
-F 2 "Connector_Molex:Molex_KK-254_AE-6410-03A_1x03_P2.54mm_Vertical" H 5350 4200 50  0001 C CNN
-F 3 "~" H 5350 4200 50  0001 C CNN
-	1    5350 4200
-	1    0    0    -1
-$EndComp
-$Comp
-L Device:R_POT RV4
-U 1 1 60558F68
-P 6250 4700
-F 0 "RV4" H 6181 4654 50  0000 R CNN
-F 1 "R_POT" H 6181 4745 50  0000 R CNN
-F 2 "Connector_Molex:Molex_KK-254_AE-6410-03A_1x03_P2.54mm_Vertical" H 6250 4700 50  0001 C CNN
-F 3 "~" H 6250 4700 50  0001 C CNN
-	1    6250 4700
-	1    0    0    1
-$EndComp
-$Comp
-L Device:R_POT RV3
-U 1 1 60559849
-P 6250 4200
-F 0 "RV3" H 6181 4246 50  0000 R CNN
-F 1 "R_POT" H 6181 4155 50  0000 R CNN
-F 2 "Connector_Molex:Molex_KK-254_AE-6410-03A_1x03_P2.54mm_Vertical" H 6250 4200 50  0001 C CNN
-F 3 "~" H 6250 4200 50  0001 C CNN
-	1    6250 4200
-	1    0    0    -1
-$EndComp
-Wire Wire Line
-	5500 4200 5650 4200
-Wire Wire Line
-	5500 4700 5650 4700
-Wire Wire Line
-	6400 4700 6450 4700
-Wire Wire Line
-	6400 4200 6450 4200
+Wire Wire Line
+	5350 4850 5350 5250
+Wire Wire Line
+	3800 4450 6250 4450
+Wire Wire Line
+	5350 3650 5350 4050
+Wire Wire Line
+	5350 4050 6250 4050
+Wire Wire Line
+	5350 4850 6250 4850
+$Comp
+L Device:R R10
+U 1 1 6124207F
+P 3050 5000
+F 0 "R10" H 3120 5046 50  0000 L CNN
+F 1 "1M_DNP" H 3120 4955 50  0000 L CNN
+F 2 "Resistor_THT:R_Axial_DIN0207_L6.3mm_D2.5mm_P10.16mm_Horizontal" V 2980 5000 50  0001 C CNN
+F 3 "~" H 3050 5000 50  0001 C CNN
+	1    3050 5000
+	1    0    0    -1
+$EndComp
+$Comp
+L Device:R R9
+U 1 1 6124278B
+P 3050 3900
+F 0 "R9" H 3120 3946 50  0000 L CNN
+F 1 "1M_DNP" H 3120 3855 50  0000 L CNN
+F 2 "Resistor_THT:R_Axial_DIN0207_L6.3mm_D2.5mm_P10.16mm_Horizontal" V 2980 3900 50  0001 C CNN
+F 3 "~" H 3050 3900 50  0001 C CNN
+	1    3050 3900
+	1    0    0    -1
+$EndComp
+Wire Wire Line
+	3050 3750 3050 3550
+Connection ~ 3050 3550
+Wire Wire Line
+	3050 3550 2350 3550
+Wire Wire Line
+	3050 4050 3050 4450
+Connection ~ 3050 4450
+Wire Wire Line
+	3050 4450 3550 4450
+Wire Wire Line
+	3050 5150 3050 5350
+Connection ~ 3050 5350
+Wire Wire Line
+	3050 5350 3250 5350
+Wire Wire Line
+	3050 4850 3050 4450
+$Comp
+L Device:R_POT_Dual RV1
+U 1 1 6125A0A4
+P 6350 4450
+F 0 "RV1" V 6304 4263 50  0000 R CNN
+F 1 "R_POT_Dual" V 6395 4263 50  0000 R CNN
+F 2 "Potentiometer_THT:Potentiometer_Alpha_RD902F-40-00D_Dual_Vertical" H 6600 4375 50  0001 C CNN
+F 3 "~" H 6600 4375 50  0001 C CNN
+	1    6350 4450
+	0    1    1    0
+$EndComp
+Wire Wire Line
+	6450 4200 6450 4100
+$Comp
+L Device:R R21
+U 1 1 61285D2E
+P 6450 3950
+F 0 "R21" H 6520 3996 50  0000 L CNN
+F 1 "150" H 6520 3905 50  0000 L CNN
+F 2 "Resistor_THT:R_Axial_DIN0207_L6.3mm_D2.5mm_P10.16mm_Horizontal" V 6380 3950 50  0001 C CNN
+F 3 "~" H 6450 3950 50  0001 C CNN
+	1    6450 3950
+	-1   0    0    1
+$EndComp
+$Comp
+L Device:R R22
+U 1 1 61286611
+P 6450 4950
+F 0 "R22" H 6520 4996 50  0000 L CNN
+F 1 "150" H 6520 4905 50  0000 L CNN
+F 2 "Resistor_THT:R_Axial_DIN0207_L6.3mm_D2.5mm_P10.16mm_Horizontal" V 6380 4950 50  0001 C CNN
+F 3 "~" H 6450 4950 50  0001 C CNN
+	1    6450 4950
+	-1   0    0    1
+$EndComp
+Wire Wire Line
+	6450 5100 6650 5100
+Connection ~ 6650 5100
+Wire Wire Line
+	6650 5100 6650 5350
+Wire Wire Line
+	6450 3800 6650 3800
+Connection ~ 6650 3800
+Wire Wire Line
+	6650 3800 6650 3550
 $EndSCHEMATC
